File: hardware/rtc.kicad_pcb (KiCad board)
At the start: 2 copper layers, 25 x 25 mm, 28 parts, among them P1 CON-SENSOR, P2 Debug, P3 Boot, U1 XMC1XXX24, U2 PCF85263AT, U3 DRILL, U4 DRILL, U5 DRILL, U6 DRILL, X1 32.768kHz

Commit message: fix ce logo orientation
Parts:
- turned VAL to 0 degrees
Changed lines of the file:
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@@
     (links 55)
     (no_connects 0)
-    (area 125.109499 87.909499 150.490501 113.290501)
+    (area 124.445139 87.245139 282.795857 162.890793)
     (thickness 1.6002)
     (drawings 12)
@@
   )
   (layers
-    (0 Vorderseite signal hide)
+    (0 Vorderseite signal)
     (31 Rückseite signal hide)
     (32 B.Adhes user)
@@
   )
   (setup
-    (last_trace_width 0.2)
+    (last_trace_width 0.249)
     (user_trace_width 0.2)
     (user_trace_width 0.25)
@@
     (aux_axis_origin 125.3 113.1)
     (grid_origin 125.3 113.1)
-    (visible_elements FFFF7FFF)
+    (visible_elements FFFFFFFF)
     (pcbplotparams
       (layerselection 0x010c8_00000001)
@@
   )
   (module kicad-libraries:CE_5mm (layer Rückseite)
-    (at 137.8 104.6 180)
-    (fp_text reference VAL (at 0 0 180) (layer B.SilkS) hide
+    (at 137.8 104.6)
+    (fp_text reference VAL (at 0 0) (layer B.SilkS) hide
       (effects (font (size 0.2 0.2) (thickness 0.05)) (justify mirror))
     )
-    (fp_text value CE_5mm (at 0 0 180) (layer B.SilkS) hide
+    (fp_text value CE_5mm (at 0 0) (layer B.SilkS) hide
       (effects (font (size 0.2 0.2) (thickness 0.05)) (justify mirror))
     )

Commit message: fix weee logo
Parts:
- VAL: footprint kicad-libraries:WEEE_7mm_back -> kicad-libraries:WEEE_7mm
- turned VAL to 0 degrees

Commit message: specify processor
Parts:
- U1: value XMC1XXX24 -> XMC1100
Changed lines of the file:
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@@
     (aux_axis_origin 125.3 113.1)
     (grid_origin 125.3 113.1)
-    (visible_elements FFFFBFFF)
+    (visible_elements FFFF7FFF)
     (pcbplotparams
       (layerselection 0x010c8_00000001)
@@
       (effects (font (size 0.3 0.3) (thickness 0.075)))
     )
-    (fp_text value XMC1XXX24 (at 0 0.8) (layer F.Fab)
+    (fp_text value XMC1100 (at 0 0.8) (layer F.Fab)
       (effects (font (size 0.3 0.3) (thickness 0.075)))
     )
